Commit message: Halfway through project

File: Level2/ros2_ws/src/my_robot_description/urdf/common_properties.xacro (robot description, xacro)
@@ -4,9 +4,15 @@
         <color rgba="0.7 0 0 1" />
     </material>
-        <material name="green">
+    <material name="green">
         <color rgba="0 0.7 0 1" />
     </material>
-        <material name="blue">
+    <material name="blue">
         <color rgba="0 0 0.7 1" />
+    </material>
+    <material name="orange">
+        <color rgba="1 0.4 0 1" />
+    </material>
+    <material name="yellow">
+        <color rgba="0.85 0.85 0 1" />
     </material>
     <xacro:macro name="box_inertia" params="l w h m xyz rpy" >

File: Level2/ros2_ws/src/my_robot_description/urdf/mobile_base.xacro (robot description, xacro)
@@ -1,4 +1,9 @@
 <?xml version="1.0"?>
 <robot xmlns:xacro="http://www.ros.org/wiki/xacro" >
+    <xacro:property name="base_length" value="0.6" />
+    <xacro:property name="base_width" value="0.4" />
+    <xacro:property name="base_height" value="0.2" />
+    <xacro:property name="wheel_radius" value="0.1" />
+    <xacro:property name="wheel_length" value="0.05" />
     <link name="base_footprint" />
     <link name="base_link">

File: Level2/ros2_ws/src/my_robot_description/urdf/my_robot.urdf.xacro (robot description, xacro)
@@ -1,11 +1,8 @@
 <?xml version="1.0"?>
 <robot name="myBot" xmlns:xacro="http://www.ros.org/wiki/xacro" >
-    <xacro:property name="base_length" value="0.6" />
-    <xacro:property name="base_width" value="0.4" />
-    <xacro:property name="base_height" value="0.2" />
-    <xacro:property name="wheel_radius" value="0.1" />
-    <xacro:property name="wheel_length" value="0.05" />
     <xacro:include filename="common_properties.xacro" />
     <xacro:include filename="mobile_base.xacro" />
+    <xacro:include filename="camera.xacro" />
     <xacro:include filename="mobile_base_gazebo.xacro" />
+    <xacro:include filename="robotic_arm.xacro" />
 </robot>
